File: siox.kicad_pcb (KiCad board)
At the start: 2 copper layers, 44.2 x 22.8 mm, 18 parts, among them J1 CE, J10 M7, J2 CI, J3 XE, J4 XI, J5 M2, J6 M3, J7 M4, J8 M5, J9 M6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

Commit message: update
Parts:
- moved J3 0.61 mm to (118.4, 70.0), turned to 180 degrees
- turned J1 to 90 degrees
- turned J2 to -90 degrees
Changed lines of the file:
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@@
   (net 15 "P12")
   (footprint "TestPoint:TestPoint_Pad_D2.0mm" (layer "F.Cu")
-    (at 121.65 61.95)
-    (descr "SMD pad as test Point, diameter 2.0mm")
-    (tags "test point SMD pad")
-    (property "Sheetfile" "siox.kicad_sch")
-    (property "Sheetname" "")
-    (property "ki_description" "Generic connector, single row, 01x01, script generated (kicad-library-utils/schlib/autogen/connector/)")
-    (property "ki_keywords" "connector")
-    (fp_text reference "J1" (at 0 -1.998) (layer "F.SilkS") hide
-        (effects (font (size 1 1) (thickness 0.15)))
-    )
-    (fp_text value "CE" (at -0.2 -2.05) (layer "F.SilkS")
-        (effects (font (size 1 1) (thickness 0.15)))
-    )
-    (fp_text user "${REFERENCE}" (at 0 -2) (layer "F.Fab")
-        (effects (font (size 1 1) (thickness 0.15)))
-    )
-    (fp_circle (center 0 0) (end 0 1.2)
-      (stroke (width 0.12) (type solid)) (fill none) (layer "F.SilkS"))
-    (fp_circle (center 0 0) (end 1.5 0)
-      (stroke (width 0.05) (type solid)) (fill none) (layer "F.CrtYd"))
-    (pad "1" smd circle (at 0 0) (size 2 2) (layers "F.Cu" "F.Mask")
+    (at 121.65 61.95 90)
+    (descr "SMD pad as test Point, diameter 2.0mm")
+    (tags "test point SMD pad")
+    (property "Sheetfile" "siox.kicad_sch")
+    (property "Sheetname" "")
+    (property "ki_description" "Generic connector, single row, 01x01, script generated (kicad-library-utils/schlib/autogen/connector/)")
+    (property "ki_keywords" "connector")
+    (fp_text reference "J1" (at 0 -1.998 90) (layer "F.SilkS") hide
+        (effects (font (size 1 1) (thickness 0.15)))
+    )
+    (fp_text value "CE" (at -0.2 -2.05 90) (layer "F.SilkS")
+        (effects (font (size 1 1) (thickness 0.15)))
+    )
+    (fp_text user "${REFERENCE}" (at 0 -2 90) (layer "F.Fab")
+        (effects (font (size 1 1) (thickness 0.15)))
+    )
+    (fp_circle (center 0 0) (end 0 1.2)
+      (stroke (width 0.12) (type solid)) (fill none) (layer "F.SilkS"))
+    (fp_circle (center 0 0) (end 1.5 0)
+      (stroke (width 0.05) (type solid)) (fill none) (layer "F.CrtYd"))
+    (pad "1" smd circle (at 0 0 90) (size 2 2) (layers "F.Cu" "F.Mask")
       (net 5 "CE") (pinfunction "Pin_1") (pintype "passive"))
   )
@@
   )
   (footprint "TestPoint:TestPoint_Pad_D2.0mm" (layer "F.Cu")
-    (at 118.5 69.45)
+    (at 118.4 70.05 180)
     (descr "SMD pad as test Point, diameter 2.0mm")
     (tags "test point SMD pad")
@@
     (fp_circle (center 0 0) (end 1.5 0)
       (stroke (width 0.05) (type solid)) (fill none) (layer "F.CrtYd"))
-    (pad "1" smd circle (at 0 0) (size 2 2) (layers "F.Cu" "F.Mask")
+    (pad "1" smd circle (at 0 0 180) (size 2 2) (layers "F.Cu" "F.Mask")
       (net 13 "P2") (pinfunction "Pin_1") (pintype "passive"))
   )
@@
   )
   (footprint "TestPoint:TestPoint_Pad_D2.0mm" (layer "F.Cu")
-    (at 121.65 65.2)
-    (descr "SMD pad as test Point, diameter 2.0mm")
-    (tags "test point SMD pad")
-    (property "Sheetfile" "siox.kicad_sch")
-    (property "Sheetname" "")
-    (property "ki_description" "Generic connector, single row, 01x01, script generated (kicad-library-utils/schlib/autogen/connector/)")
-    (property "ki_keywords" "connector")
-    (fp_text reference "J2" (at 0 -1.998) (layer "F.SilkS") hide
-        (effects (font (size 1 1) (thickness 0.15)))
-    )
-    (fp_text value "CI" (at 0 2.05) (layer "F.SilkS")
-        (effects (font (size 1 1) (thickness 0.15)))
-    )
-    (fp_text user "${REFERENCE}" (at 0 -2) (layer "F.Fab")
-        (effects (font (size 1 1) (thickness 0.15)))
-    )
-    (fp_circle (center 0 0) (end 0 1.2)
-      (stroke (width 0.12) (type solid)) (fill none) (layer "F.SilkS"))
-    (fp_circle (center 0 0) (end 1.5 0)
-      (stroke (width 0.05) (type solid)) (fill none) (layer "F.CrtYd"))
-    (pad "1" smd circle (at 0 0) (size 2 2) (layers "F.Cu" "F.Mask")
+    (at 121.65 65.2 -90)
+    (descr "SMD pad as test Point, diameter 2.0mm")
+    (tags "test point SMD pad")
+    (property "Sheetfile" "siox.kicad_sch")
+    (property "Sheetname" "")
+    (property "ki_description" "Generic connector, single row, 01x01, script generated (kicad-library-utils/schlib/autogen/connector/)")
+    (property "ki_keywords" "connector")
+    (fp_text reference "J2" (at 0 -1.998 90) (layer "F.SilkS") hide
+        (effects (font (size 1 1) (thickness 0.15)))
+    )
+    (fp_text value "CI" (at 0 2.05 90) (layer "F.SilkS")
+        (effects (font (size 1 1) (thickness 0.15)))
+    )
+    (fp_text user "${REFERENCE}" (at 0 -2 90) (layer "F.Fab")
+        (effects (font (size 1 1) (thickness 0.15)))
+    )
+    (fp_circle (center 0 0) (end 0 1.2)
+      (stroke (width 0.12) (type solid)) (fill none) (layer "F.SilkS"))
+    (fp_circle (center 0 0) (end 1.5 0)
+      (stroke (width 0.05) (type solid)) (fill none) (layer "F.CrtYd"))
+    (pad "1" smd circle (at 0 0 270) (size 2 2) (layers "F.Cu" "F.Mask")
       (net 4 "CI") (pinfunction "Pin_1") (pintype "passive"))
   )
@@
   (segment (start 108 71) (end 106 69) (width 0.25) (layer "F.Cu") (net 12))
   (segment (start 104.45 69) (end 100.265 64.815) (width 0.25) (layer "F.Cu") (net 12))
-  (segment (start 107.8 64.05) (end 111.95 68.2) (width 0.25) (layer "F.Cu") (net 13))
+  (segment (start 106 61.15) (end 106 63.459619) (width 0.25) (layer "F.Cu") (net 13))
   (segment (start 107.1375 64.05) (end 107.8 64.05) (width 0.25) (layer "F.Cu") (net 13))
-  (segment (start 106 61.15) (end 106 63.459619) (width 0.25) (layer "F.Cu") (net 13))
-  (segment (start 117.25 68.2) (end 118.5 69.45) (width 0.25) (layer "F.Cu") (net 13))
+  (segment (start 116.55 68.2) (end 118.4 70.05) (width 0.25) (layer "F.Cu") (net 13))
   (segment (start 105.838 59.7375) (end 105.95 59.6255) (width 0.25) (layer "F.Cu") (net 13))
-  (segment (start 111.95 68.2) (end 117.25 68.2) (width 0.25) (layer "F.Cu") (net 13))
+  (segment (start 111.95 68.2) (end 116.55 68.2) (width 0.25) (layer "F.Cu") (net 13))
   (segment (start 106.590381 64.05) (end 107.1375 64.05) (width 0.25) (layer "F.Cu") (net 13))
   (segment (start 104.05 59.7375) (end 105.838 59.7375) (width 0.25) (layer "F.Cu") (net 13))
   (segment (start 106.5375 64.05) (end 107.1375 64.05) (width 0.25) (layer "F.Cu") (net 13))
   (segment (start 106 63.459619) (end 106.590381 64.05) (width 0.25) (layer "F.Cu") (net 13))
+  (segment (start 107.8 64.05) (end 111.95 68.2) (width 0.25) (layer "F.Cu") (net 13))
   (via (at 106 61.15) (size 0.8) (drill 0.4) (layers "F.Cu" "B.Cu") (net 13))
   (via (at 105.95 59.6255) (size 0.8) (drill 0.4) (layers "F.Cu" "B.Cu") (net 13))

Commit message: update
Other:
- board size 44.2 x 22.8 mm -> 45 x 22.7 mm
Changed lines of the file:
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@@
     )
   )
-  (gr_line (start 90.95 50) (end 132.3 50)
-    (stroke (width 0.1) (type default)) (layer "Edge.Cuts"))
-  (gr_line (start 91.075 72.75) (end 89.3 71)
-    (stroke (width 0.1) (type default)) (layer "Edge.Cuts"))
-  (gr_line (start 111.75 69.8) (end 108.85 72.75)
-    (stroke (width 0.1) (type default)) (layer "Edge.Cuts"))
-  (gr_line (start 89.3 51.55) (end 90.95 50)
-    (stroke (width 0.1) (type default)) (layer "Edge.Cuts"))
-  (gr_line (start 133.5 58.2) (end 130.4 61.25)
-    (stroke (width 0.1) (type default)) (layer "Edge.Cuts"))
-  (gr_line (start 133.5 51.2) (end 133.5 58.2)
+  (gr_line (start 90.7 50) (end 132.7 50)
+    (stroke (width 0.1) (type default)) (layer "Edge.Cuts"))
+  (gr_line (start 90.6875 72.7) (end 88.9125 70.975)
+    (stroke (width 0.1) (type default)) (layer "Edge.Cuts"))
+  (gr_line (start 111.75 69.8) (end 108.95 72.7)
+    (stroke (width 0.1) (type default)) (layer "Edge.Cuts"))
+  (gr_line (start 88.9125 51.8) (end 90.7 50)
+    (stroke (width 0.1) (type default)) (layer "Edge.Cuts"))
+  (gr_line (start 133.9 58.2) (end 130.8 61.25)
+    (stroke (width 0.1) (type default)) (layer "Edge.Cuts"))
+  (gr_line (start 133.9 51.2) (end 133.9 58.2)
     (stroke (width 0.1) (type default)) (layer "Edge.Cuts"))
   (gr_line (start 123.75 69.5) (end 121.5 71.75)
@@
   (gr_line (start 125.25 61.25) (end 123.75 62.75)
     (stroke (width 0.1) (type default)) (layer "Edge.Cuts"))
-  (gr_line (start 130.4 61.25) (end 125.25 61.25)
-    (stroke (width 0.1) (type default)) (layer "Edge.Cuts"))
-  (gr_line (start 132.3 50) (end 133.5 51.2)
-    (stroke (width 0.1) (type default)) (layer "Edge.Cuts"))
-  (gr_line (start 108.85 72.75) (end 91.075 72.75)
+  (gr_line (start 130.8 61.25) (end 125.25 61.25)
+    (stroke (width 0.1) (type default)) (layer "Edge.Cuts"))
+  (gr_line (start 132.7 50) (end 133.9 51.2)
+    (stroke (width 0.1) (type default)) (layer "Edge.Cuts"))
+  (gr_line (start 108.95 72.7) (end 90.6875 72.7)
     (stroke (width 0.1) (type default)) (layer "Edge.Cuts"))
   (gr_line (start 123.75 62.75) (end 123.75 69.5)
     (stroke (width 0.1) (type default)) (layer "Edge.Cuts"))
-  (gr_line (start 114.85 69.8) (end 111.75 69.8)
-    (stroke (width 0.1) (type default)) (layer "Edge.Cuts"))
-  (gr_line (start 89.3 71) (end 89.3 51.55)
-    (stroke (width 0.1) (type default)) (layer "Edge.Cuts"))
-  (gr_line (start 121.5 71.75) (end 116.8 71.75)
-    (stroke (width 0.1) (type default)) (layer "Edge.Cuts"))
-  (gr_line (start 116.8 71.75) (end 114.85 69.8)
+  (gr_line (start 113.85 69.8) (end 111.75 69.8)
+    (stroke (width 0.1) (type default)) (layer "Edge.Cuts"))
+  (gr_line (start 88.9125 70.975) (end 88.9125 51.8)
+    (stroke (width 0.1) (type default)) (layer "Edge.Cuts"))
+  (gr_line (start 121.5 71.75) (end 115.75 71.75)
+    (stroke (width 0.1) (type default)) (layer "Edge.Cuts"))
+  (gr_line (start 115.75 71.75) (end 113.85 69.8)
     (stroke (width 0.1) (type default)) (layer "Edge.Cuts"))
   (gr_text "sio-x djvs" (at 122 60.45) (layer "F.SilkS")
@@
   (segment (start 107.1375 66) (end 105.8 66) (width 0.25) (layer "F.Cu") (net 15))
   (segment (start 111.1 64.7) (end 110.4755 65.3245) (width 0.25) (layer "F.Cu") (net 15))
-  (segment (start 98.35 60.25) (end 96.8625 60.25) (width 0.25) (layer "F.Cu") (net 15))
   (segment (start 96.8625 60.25) (end 96.8625 58.8025) (width 0.25) (layer "F.Cu") (net 15))
   (segment (start 105.75 66) (end 103.25 66) (width 0.25) (layer "F.Cu") (net 15))
   (segment (start 105.8 66) (end 105.75 66) (width 0.25) (layer "F.Cu") (net 15))
   (segment (start 112.8625 64.7) (end 112.8625 64.65) (width 0.25) (layer "F.Cu") (net 15))
+  (segment (start 98.05 60.8) (end 97.5 60.25) (width 0.25) (layer "F.Cu") (net 15))
   (segment (start 96.8625 58.8025) (end 95.54 57.48) (width 0.25) (layer "F.Cu") (net 15))
+  (segment (start 97.5 60.25) (end 96.8625 60.25) (width 0.25) (layer "F.Cu") (net 15))
   (segment (start 107.1375 66) (end 107.1375 66.65) (width 0.25) (layer "F.Cu") (net 15))
   (segment (start 103.25 66) (end 101.2 63.95) (width 0.25) (layer "F.Cu") (net 15))
   (segment (start 112.8625 64.05) (end 112.8625 64.7) (width 0.25) (layer "F.Cu") (net 15))
   (via (at 105.8 66) (size 0.8) (drill 0.4) (layers "F.Cu" "B.Cu") (net 15))
-  (via (at 98.35 60.25) (size 0.8) (drill 0.4) (layers "F.Cu" "B.Cu") (net 15))
+  (via (at 98.05 60.8) (size 0.8) (drill 0.4) (layers "F.Cu" "B.Cu") (net 15))
   (via (at 101.2 63.95) (size 0.8) (drill 0.4) (layers "F.Cu" "B.Cu") (net 15))
   (via (at 95.54 57.48) (size 1.66) (drill 1.02) (layers "F.Cu" "B.Cu") (free) (net 15))
   (via (at 110.4755 65.3245) (size 0.8) (drill 0.4) (layers "F.Cu" "B.Cu") (net 15))
   (segment (start 109.8 66) (end 110.4755 65.3245) (width 0.25) (layer "B.Cu") (net 15))
-  (segment (start 98.35 61.1) (end 98.35 60.25) (width 0.25) (layer "B.Cu") (net 15))
+  (segment (start 98.05 60.8) (end 101.2 63.95) (width 0.25) (layer "B.Cu") (net 15))
   (segment (start 105.8 66) (end 109.8 66) (width 0.25) (layer "B.Cu") (net 15))
-  (segment (start 101.2 63.95) (end 98.35 61.1) (width 0.25) (layer "B.Cu") (net 15))
   (zone (net 14) (net_name "GND1") (layer "F.Cu") (name "FRONTFILL") (hatch edge 0.508)
     (connect_pads (clearance 0.508))
@@
     (polygon
       (pts
-        (xy 145 45)
-        (xy 145 90)
-        (xy 85 90)
-        (xy 85 45)
+        (xy 135 49)
+        (xy 135 74)
+        (xy 88 74)
+        (xy 88 49)
       )
     )
@@
     (polygon
       (pts
-        (xy 145 45)
-        (xy 115 45)
-        (xy 85 45)
-        (xy 85 90)
-        (xy 145 90)
+        (xy 136 48)
+        (xy 115 48)
+        (xy 87 48)
+        (xy 87 75)
+        (xy 136 75)
       )
     )

Commit message: cleanup
Connections:
- net P11 renamed XI
- net P2 renamed XE
- net P8 renamed PI
Routing:
- net MP2: track 9.21 -> 8.32 mm
- net MP7: track 11.2 -> 12.0 mm
- net CE: track 29.9 -> 29.2 mm
- net GND1: track 14.0 -> 14.7 mm, vias 8 -> 38
- net CI: track 12.2 -> 11.7 mm

Commit message: updates
Other:
- board size 45 x 22.7 mm -> 45.8 x 24.1 mm
Changed lines of the file:
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@@
       (outputformat 1)
       (mirror false)
-      (drillshape 1)
+      (drillshape 0)
       (scaleselection 1)
-      (outputdirectory "")
+      (outputdirectory "outputs/gerber/")
     )
   )
@@
     (fp_line (start 1 0.625) (end -1 0.625)
       (stroke (width 0.1) (type solid)) (layer "F.Fab"))
-    (pad "1" smd roundrect (at -0.9125 0 270) (size 1.025 1.4) (layers "F.Cu" "F.Paste" "F.Mask") (roundrect_rratio 0.243902)
+    (pad "1" smd roundrect (at -0.9125 0 270) (size 1.025 1.4) (layers "F.Cu" "F.Paste" "F.Mask") (roundrect_rratio 0.243902439)
       (net 4 "MP1") (pintype "passive"))
-    (pad "2" smd roundrect (at 0.9125 0 270) (size 1.025 1.4) (layers "F.Cu" "F.Paste" "F.Mask") (roundrect_rratio 0.243902)
+    (pad "2" smd roundrect (at 0.9125 0 270) (size 1.025 1.4) (layers "F.Cu" "F.Paste" "F.Mask") (roundrect_rratio 0.243902439)
       (net 1 "P3") (pintype "passive"))
     (model "${KICAD6_3DMODEL_DIR}/Resistor_SMD.3dshapes/R_0805_2012Metric.wrl"
@@
     (fp_line (start 1 0.625) (end -1 0.625)
       (stroke (width 0.1) (type solid)) (layer "F.Fab"))
-    (pad "1" smd roundrect (at -0.9125 0 90) (size 1.025 1.4) (layers "F.Cu" "F.Paste" "F.Mask") (roundrect_rratio 0.243902)
+    (pad "1" smd roundrect (at -0.9125 0 90) (size 1.025 1.4) (layers "F.Cu" "F.Paste" "F.Mask") (roundrect_rratio 0.243902439)
       (net 2 "CI") (pintype "passive"))
-    (pad "2" smd roundrect (at 0.9125 0 90) (size 1.025 1.4) (layers "F.Cu" "F.Paste" "F.Mask") (roundrect_rratio 0.243902)
+    (pad "2" smd roundrect (at 0.9125 0 90) (size 1.025 1.4) (layers "F.Cu" "F.Paste" "F.Mask") (roundrect_rratio 0.243902439)
       (net 4 "MP1") (pintype "passive"))
     (model "${KICAD6_3DMODEL_DIR}/Resistor_SMD.3dshapes/R_0805_2012Metric.wrl"
@@
     (fp_line (start 1 0.625) (end -1 0.625)
       (stroke (width 0.1) (type solid)) (layer "F.Fab"))
-    (pad "1" smd roundrect (at -0.9125 0 180) (size 1.025 1.4) (layers "F.Cu" "F.Paste" "F.Mask") (roundrect_rratio 0.243902)
+    (pad "1" smd roundrect (at -0.9125 0 180) (size 1.025 1.4) (layers "F.Cu" "F.Paste" "F.Mask") (roundrect_rratio 0.243902439)
       (net 12 "P12") (pintype "passive"))
-    (pad "2" smd roundrect (at 0.9125 0 180) (size 1.025 1.4) (layers "F.Cu" "F.Paste" "F.Mask") (roundrect_rratio 0.243902)
+    (pad "2" smd roundrect (at 0.9125 0 180) (size 1.025 1.4) (layers "F.Cu" "F.Paste" "F.Mask") (roundrect_rratio 0.243902439)
       (net 11 "GND1") (pintype "passive"))
     (model "${KICAD6_3DMODEL_DIR}/Resistor_SMD.3dshapes/R_0805_2012Metric.wrl"
@@
     (fp_line (start 1 0.625) (end -1 0.625)
       (stroke (width 0.1) (type solid)) (layer "F.Fab"))
-    (pad "1" smd roundrect (at -0.9125 0 270) (size 1.025 1.4) (layers "F.Cu" "F.Paste" "F.Mask") (roundrect_rratio 0.243902)
+    (pad "1" smd roundrect (at -0.9125 0 270) (size 1.025 1.4) (layers "F.Cu" "F.Paste" "F.Mask") (roundrect_rratio 0.243902439)
       (net 13 "XE") (pintype "passive"))
-    (pad "2" smd roundrect (at 0.9125 0 270) (size 1.025 1.4) (layers "F.Cu" "F.Paste" "F.Mask") (roundrect_rratio 0.243902)
+    (pad "2" smd roundrect (at 0.9125 0 270) (size 1.025 1.4) (layers "F.Cu" "F.Paste" "F.Mask") (roundrect_rratio 0.243902439)
       (net 4 "MP1") (pintype "passive"))
     (model "${KICAD6_3DMODEL_DIR}/Resistor_SMD.3dshapes/R_0805_2012Metric.wrl"
@@
     )
   )
-  (gr_line (start 90.7 50) (end 132.7 50)
-    (stroke (width 0.1) (type default)) (layer "Edge.Cuts"))
-  (gr_line (start 90.6875 72.7) (end 88.9125 70.975)
-    (stroke (width 0.1) (type default)) (layer "Edge.Cuts"))
-  (gr_line (start 111.75 69.8) (end 108.95 72.7)
-    (stroke (width 0.1) (type default)) (layer "Edge.Cuts"))
-  (gr_line (start 88.9125 51.8) (end 90.7 50)
-    (stroke (width 0.1) (type default)) (layer "Edge.Cuts"))
-  (gr_line (start 133.9 58.2) (end 130.8 61.25)
-    (stroke (width 0.1) (type default)) (layer "Edge.Cuts"))
-  (gr_line (start 133.9 51.2) (end 133.9 58.2)
-    (stroke (width 0.1) (type default)) (layer "Edge.Cuts"))
-  (gr_line (start 123.75 69.5) (end 121.5 71.75)
-    (stroke (width 0.1) (type default)) (layer "Edge.Cuts"))
-  (gr_line (start 125.25 61.25) (end 123.75 62.75)
-    (stroke (width 0.1) (type default)) (layer "Edge.Cuts"))
-  (gr_line (start 130.8 61.25) (end 125.25 61.25)
-    (stroke (width 0.1) (type default)) (layer "Edge.Cuts"))
-  (gr_line (start 132.7 50) (end 133.9 51.2)
-    (stroke (width 0.1) (type default)) (layer "Edge.Cuts"))
-  (gr_line (start 108.95 72.7) (end 90.6875 72.7)
-    (stroke (width 0.1) (type default)) (layer "Edge.Cuts"))
-  (gr_line (start 123.75 62.75) (end 123.75 69.5)
-    (stroke (width 0.1) (type default)) (layer "Edge.Cuts"))
-  (gr_line (start 113.85 69.8) (end 111.75 69.8)
-    (stroke (width 0.1) (type default)) (layer "Edge.Cuts"))
-  (gr_line (start 88.9125 70.975) (end 88.9125 51.8)
-    (stroke (width 0.1) (type default)) (layer "Edge.Cuts"))
-  (gr_line (start 121.5 71.75) (end 115.75 71.75)
-    (stroke (width 0.1) (type default)) (layer "Edge.Cuts"))
-  (gr_line (start 115.75 71.75) (end 113.85 69.8)
+  (gr_arc (start 124.6 63.8) (mid 125.273654 62.173654) (end 126.9 61.5)
+    (stroke (width 0.1) (type default)) (layer "Edge.Cuts"))
+  (gr_line (start 133.973654 51.6) (end 133.973654 59.2)
+    (stroke (width 0.1) (type default)) (layer "Edge.Cuts"))
+  (gr_arc (start 133.973654 59.2) (mid 133.3 60.826346) (end 131.673654 61.5)
+    (stroke (width 0.1) (type default)) (layer "Edge.Cuts"))
+  (gr_line (start 131.673654 61.5) (end 126.9 61.5)
+    (stroke (width 0.1) (type default)) (layer "Edge.Cuts"))
+  (gr_line (start 124.6 63.8) (end 124.6 71.1)
+    (stroke (width 0.1) (type default)) (layer "Edge.Cuts"))
+  (gr_arc (start 131.673654 49.3) (mid 133.3 49.973654) (end 133.973654 51.6)
+    (stroke (width 0.1) (type default)) (layer "Edge.Cuts"))
+  (gr_line (start 90.626346 49.326346) (end 131.673654 49.3)
+    (stroke (width 0.1) (type default)) (layer "Edge.Cuts"))
+  (gr_arc (start 124.6 71.1) (mid 123.926346 72.726346) (end 122.3 73.4)
+    (stroke (width 0.1) (type default)) (layer "Edge.Cuts"))
+  (gr_line (start 88.126346 51.826346) (end 88.126346 71.1)
+    (stroke (width 0.1) (type default)) (layer "Edge.Cuts"))
+  (gr_arc (start 111.6 71.1) (mid 113.3 69.4) (end 115 71.1)
+    (stroke (width 0.1) (type default)) (layer "Edge.Cuts"))
+  (gr_arc (start 111.6 71.1) (mid 110.926346 72.726346) (end 109.3 73.4)
+    (stroke (width 0.1) (type default)) (layer "Edge.Cuts"))
+  (gr_arc (start 117.3 73.4) (mid 115.673654 72.726346) (end 115 71.1)
+    (stroke (width 0.1) (type default)) (layer "Edge.Cuts"))
+  (gr_line (start 122.3 73.4) (end 117.3 73.4)
+    (stroke (width 0.1) (type default)) (layer "Edge.Cuts"))
+  (gr_arc (start 88.126346 51.826346) (mid 88.858579 50.058579) (end 90.626346 49.326346)
+    (stroke (width 0.1) (type default)) (layer "Edge.Cuts"))
+  (gr_arc (start 90.426346 73.4) (mid 88.8 72.726346) (end 88.126346 71.1)
+    (stroke (width 0.1) (type default)) (layer "Edge.Cuts"))
+  (gr_line (start 109.3 73.4) (end 90.426346 73.4)
     (stroke (width 0.1) (type default)) (layer "Edge.Cuts"))
   (gr_text "sio-x djvs" (at 122 60.45) (layer "F.SilkS")

Commit message: fix pads
Parts:
- added J11: IO_GND_1, PsioPin:PsioPin, F.Cu at (132.4, 51.8)
- added J12: IO_GND_2, PsioPin:PsioPin, F.Cu at (90.5, 53.7)
- added J13: IO_GND_3, PsioPin:PsioPin, F.Cu at (90.5, 57.5)
- added J14: IO_GND_4, PsioPin:PsioPin, F.Cu at (132.4, 55.6)
- added J15: IO_CE, PsioPin:PsioPin, F.Cu at (128.6, 53.7)
- added J16: IO_PI, PsioPin:PsioPin, F.Cu at (128.6, 57.5)
- added J17: M7, PsioPin:PsioPin, F.Cu at (110.8, 53.7)
- added J18: M7, PsioPin:PsioPin, F.Cu at (110.8, 57.5)
- added J19: IO_PI, PsioPin:PsioPin, F.Cu at (95.5, 57.5)
Connections:
- net P12 renamed EN
Routing:
- net GND1: track 14.7 -> 18.5 mm, vias 38 -> 34
- net PI: vias 2 -> 1
- net MP1: vias 2 -> 0
- net EN: vias 5 -> 4
- net CE: vias 3 -> 2

Commit message: updates
Parts:
- J15: value IO_CE -> IO_PE
- moved J10 1.45 mm to (109.5, 70.9)
- moved J5 1.05 mm to (90.7, 70.9)
- moved J4 1.00 mm to (121.7, 69.5)
- moved J9 0.95 mm to (105.7, 70.9)
- moved J3 0.72 mm to (118.1, 70.7)
- moved J6 0.56 mm to (94.5, 70.9)
- moved J2 0.50 mm to (121.7, 65.7)
- moved J8 0.46 mm to (102.0, 70.9)
- moved J7 0.09 mm to (98.2, 70.9)
Routing:
- net GND1: track 18.5 -> 16.9 mm, vias 34 -> 24
- net MP3: track 9.66 -> 8.45 mm
- net MP7: track 12.0 -> 12.6 mm
- net P3: track 8.06 -> 8.59 mm
- net MP2: track 8.32 -> 7.81 mm
