File: siox.kicad_pcb (KiCad board)
At the start: 2 copper layers, 45.8 x 24.1 mm, 27 parts, among them J1 CE, J10 M7, J11 IO_GND_1, J12 IO_GND_2, J13 IO_GND_3, J14 IO_GND_4, J15 IO_PE, J16 IO_PI, J17 M7, J18 M7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

Commit message: updates
Connections:
- R2 pad 2: P3 -> P13
- U1 pad 12: EN -> P12
- U1 pad 13: EN -> P13
- U1 pad 3: P3 -> P13
Routing:
- net P13: track 0.00 -> 15.4 mm, vias 0 -> 2
- net P3: track 8.59 -> 0.00 mm
- net EN: track 24.9 -> 16.6 mm, vias 4 -> 3
- net GND1: track 16.9 -> 18.7 mm, vias 24 -> 25
- net XE: track 21.5 -> 22.3 mm
Changed lines of the file:
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@@
   )
   (net 0 "")
-  (net 1 "P3")
+  (net 1 "P13")
   (net 2 "CI")
   (net 3 "CE")
@@
   (net 14 "PI")
   (net 15 "EN")
+  (net 16 "P12")
   (footprint "TestPoint:TestPoint_Pad_D2.0mm" (layer "F.Cu")
     (at 121.65 61.95 90)
@@
       (net 4 "MP1") (pintype "passive"))
     (pad "2" smd roundrect (at 0.9125 0 270) (size 1.025 1.4) (layers "F.Cu" "F.Paste" "F.Mask") (roundrect_rratio 0.243902439)
-      (net 1 "P3") (pintype "passive"))
+      (net 1 "P13") (pintype "passive"))
     (model "${KICAD6_3DMODEL_DIR}/Resistor_SMD.3dshapes/R_0805_2012Metric.wrl"
       (offset (xyz 0 0 0))
@@
       (net 12 "XE") (pinfunction "ACLK/TACLK/A0/P1.0") (pintype "bidirectional"))
     (pad "3" smd roundrect (at -2.8625 -0.65) (size 1.475 0.4) (layers "F.Cu" "F.Paste" "F.Mask") (roundrect_rratio 0.25)
-      (net 1 "P3") (pinfunction "TA0.0/A1/P1.1") (pintype "bidirectional"))
+      (net 1 "P13") (pinfunction "TA0.0/A1/P1.1") (pintype "bidirectional"))
     (pad "4" smd roundrect (at -2.8625 0) (size 1.475 0.4) (layers "F.Cu" "F.Paste" "F.Mask") (roundrect_rratio 0.25)
       (net 11 "GND1") (pinfunction "TA0.1/A2/P1.2") (pintype "bidirectional"))
@@
       (net 13 "XI") (pinfunction "SBWTCK/TEST") (pintype "input"))
     (pad "12" smd roundrect (at 2.8625 -0.65) (size 1.475 0.4) (layers "F.Cu" "F.Paste" "F.Mask") (roundrect_rratio 0.25)
-      (net 15 "EN") (pinfunction "P2.7/XOUT") (pintype "bidirectional"))
+      (net 16 "P12") (pinfunction "P2.7/XOUT") (pintype "bidirectional"))
     (pad "13" smd roundrect (at 2.8625 -1.3) (size 1.475 0.4) (layers "F.Cu" "F.Paste" "F.Mask") (roundrect_rratio 0.25)
-      (net 15 "EN") (pinfunction "P2.6/XIN/TA0.1") (pintype "bidirectional"))
+      (net 1 "P13") (pinfunction "P2.6/XIN/TA0.1") (pintype "bidirectional"))
     (pad "14" smd roundrect (at 2.8625 -1.95) (size 1.475 0.4) (layers "F.Cu" "F.Paste" "F.Mask") (roundrect_rratio 0.25)
       (net 4 "MP1") (pinfunction "DVSS") (pintype "power_in"))
@@
   (via (at 131.1 53.66) (size 1.66) (drill 1.02) (layers "F.Cu" "B.Cu") (net 0))
   (via (at 120.94 53.66) (size 1.66) (drill 1.02) (layers "F.Cu" "B.Cu") (net 0))
-  (segment (start 100.4 62.425) (end 100.558884 62.425) (width 0.25) (layer "F.Cu") (net 1))
-  (segment (start 100.4 61.5125) (end 100.4 62.425) (width 0.25) (layer "F.Cu") (net 1))
-  (segment (start 100.558884 62.425) (end 102.833884 64.7) (width 0.25) (layer "F.Cu") (net 1))
+  (segment (start 112.8625 64.7) (end 111.1 64.7) (width 0.25) (layer "F.Cu") (net 1))
+  (segment (start 111.1 64.7) (end 110.4755 65.3245) (width 0.25) (layer "F.Cu") (net 1))
+  (segment (start 107.1375 64.7) (end 108.65 64.7) (width 0.25) (layer "F.Cu") (net 1))
+  (segment (start 100.4 62.266116) (end 102.833884 64.7) (width 0.25) (layer "F.Cu") (net 1))
+  (segment (start 108.65 64.7) (end 108.725 64.775) (width 0.25) (layer "F.Cu") (net 1))
   (segment (start 102.833884 64.7) (end 107.1375 64.7) (width 0.25) (layer "F.Cu") (net 1))
+  (segment (start 100.4 61.5125) (end 100.4 62.266116) (width 0.25) (layer "F.Cu") (net 1))
+  (segment (start 112.8625 64.05) (end 112.8625 64.7) (width 0.25) (layer "F.Cu") (net 1))
+  (via (at 108.725 64.775) (size 0.8) (drill 0.4) (layers "F.Cu" "B.Cu") (net 1))
+  (via (at 110.4755 65.3245) (size 0.8) (drill 0.4) (layers "F.Cu" "B.Cu") (net 1))
+  (segment (start 108.725 64.775) (end 109.926 64.775) (width 0.25) (layer "B.Cu") (net 1))
+  (segment (start 109.926 64.775) (end 110.4755 65.3245) (width 0.25) (layer "B.Cu") (net 1))
   (segment (start 112.8625 66.65) (end 112.8625 66) (width 0.25) (layer "F.Cu") (net 2))
   (segment (start 114.95 64.7255) (end 115.387 64.7255) (width 0.25) (layer "F.Cu") (net 2))
@@
   (segment (start 100.86 66.085) (end 105.7 70.925) (width 0.25) (layer "F.Cu") (net 9))
   (segment (start 99.4 66.085) (end 100.86 66.085) (width 0.25) (layer "F.Cu") (net 9))
-  (segment (start 103.95 66.95) (end 105.025 68.025) (width 0.25) (layer "F.Cu") (net 10))
-  (segment (start 106.55 68.025) (end 109.45 70.925) (width 0.25) (layer "F.Cu") (net 10))
-  (segment (start 105.025 68.025) (end 106.55 68.025) (width 0.25) (layer "F.Cu") (net 10))
-  (segment (start 103.3 66.95) (end 103.95 66.95) (width 0.25) (layer "F.Cu") (net 10))
+  (segment (start 105.425 69.075) (end 107.6 69.075) (width 0.25) (layer "F.Cu") (net 10))
+  (segment (start 107.6 69.075) (end 109.45 70.925) (width 0.25) (layer "F.Cu") (net 10))
   (segment (start 99.4 64.815) (end 101.165 64.815) (width 0.25) (layer "F.Cu") (net 10))
-  (segment (start 101.165 64.815) (end 103.3 66.95) (width 0.25) (layer "F.Cu") (net 10))
+  (segment (start 101.165 64.815) (end 105.425 69.075) (width 0.25) (layer "F.Cu") (net 10))
   (segment (start 96.745 63.545) (end 99.4 63.545) (width 0.25) (layer "F.Cu") (net 11))
   (segment (start 95.0375 60.25) (end 95.0375 60.463) (width 0.25) (layer "F.Cu") (net 11))
   (segment (start 95.0375 60.463) (end 95.8 61.2255) (width 0.25) (layer "F.Cu") (net 11))
+  (segment (start 107.1375 67.3) (end 105.475 67.3) (width 0.25) (layer "F.Cu") (net 11))
   (segment (start 108 65.35) (end 108.8 66.15) (width 0.25) (layer "F.Cu") (net 11))
+  (segment (start 105.475 67.3) (end 105.35 67.425) (width 0.25) (layer "F.Cu") (net 11))
   (segment (start 90.46 53.66) (end 90.46 57.48) (width 0.25) (layer "F.Cu") (net 11))
   (segment (start 107.1375 67.3) (end 108.825 67.3) (width 0.25) (layer "F.Cu") (net 11))
@@
   (via (at 115.825 69.975) (size 0.8) (drill 0.4) (layers "F.Cu" "B.Cu") (free) (net 11))
   (via (at 109.55 58.925) (size 0.8) (drill 0.4) (layers "F.Cu" "B.Cu") (free) (net 11))
+  (via (at 105.35 67.425) (size 0.8) (drill 0.4) (layers "F.Cu" "B.Cu") (net 11))
   (via (at 122.125 59.975) (size 0.8) (drill 0.4) (layers "F.Cu" "B.Cu") (free) (net 11))
   (via (at 104.75 63.1) (size 0.8) (drill 0.4) (layers "F.Cu" "B.Cu") (free) (net 11))
@@
   (segment (start 95.8 61.2255) (end 95.8 62.6) (width 0.25) (layer "B.Cu") (net 11))
   (segment (start 95.8 62.6) (end 96 62.8) (width 0.25) (layer "B.Cu") (net 11))
+  (segment (start 111.95 68.2) (end 115.6 68.2) (width 0.25) (layer "F.Cu") (net 12))
+  (segment (start 109.2 64.05) (end 109.475 64.325) (width 0.25) (layer "F.Cu") (net 12))
+  (segment (start 106 61.15) (end 106 63.459619) (width 0.25) (layer "F.Cu") (net 12))
+  (segment (start 109.475 64.325) (end 109.475 65.725) (width 0.25) (layer "F.Cu") (net 12))
   (segment (start 115.6 68.2) (end 118.1 70.7) (width 0.25) (layer "F.Cu") (net 12))
-  (segment (start 106 61.15) (end 106 63.459619) (width 0.25) (layer "F.Cu") (net 12))
-  (segment (start 114.65 68.2) (end 115.6 68.2) (width 0.25) (layer "F.Cu") (net 12))
-  (segment (start 107.1375 64.05) (end 107.8 64.05) (width 0.25) (layer "F.Cu") (net 12))
+  (segment (start 107.1375 64.05) (end 109.2 64.05) (width 0.25) (layer "F.Cu") (net 12))
+  (segment (start 109.475 65.725) (end 111.95 68.2) (width 0.25) (layer "F.Cu") (net 12))
   (segment (start 105.838 59.7375) (end 105.95 59.6255) (width 0.25) (layer "F.Cu") (net 12))
   (segment (start 106.590381 64.05) (end 107.1375 64.05) (width 0.25) (layer "F.Cu") (net 12))
@@
   (segment (start 106.5375 64.05) (end 107.1375 64.05) (width 0.25) (layer "F.Cu") (net 12))
   (segment (start 106 63.459619) (end 106.590381 64.05) (width 0.25) (layer "F.Cu") (net 12))
-  (segment (start 111.95 68.2) (end 114.65 68.2) (width 0.25) (layer "F.Cu") (net 12))
-  (segment (start 107.8 64.05) (end 111.95 68.2) (width 0.25) (layer "F.Cu") (net 12))
   (via (at 106 61.15) (size 0.8) (drill 0.4) (layers "F.Cu" "B.Cu") (net 12))
   (via (at 105.95 59.6255) (size 0.8) (drill 0.4) (layers "F.Cu" "B.Cu") (net 12))
@@
   (segment (start 118.358058 62.258058) (end 121.615616 59.0005) (width 0.25) (layer "B.Cu") (net 14))
   (segment (start 128.5505 58.6) (end 128.5505 57.4895) (width 0.25) (layer "B.Cu") (net 14))
-  (segment (start 112.8625 64.7) (end 111.1 64.7) (width 0.25) (layer "F.Cu") (net 15))
-  (segment (start 107.1375 66) (end 105.8 66) (width 0.25) (layer "F.Cu") (net 15))
-  (segment (start 111.1 64.7) (end 110.4755 65.3245) (width 0.25) (layer "F.Cu") (net 15))
+  (segment (start 105.275 66) (end 103.25 66) (width 0.25) (layer "F.Cu") (net 15))
+  (segment (start 105.275 66) (end 107.1375 66) (width 0.25) (layer "F.Cu") (net 15))
   (segment (start 96.8625 60.25) (end 96.8625 58.8025) (width 0.25) (layer "F.Cu") (net 15))
-  (segment (start 105.75 66) (end 103.25 66) (width 0.25) (layer "F.Cu") (net 15))
-  (segment (start 105.8 66) (end 105.75 66) (width 0.25) (layer "F.Cu") (net 15))
   (segment (start 98.05 60.8) (end 97.5 60.25) (width 0.25) (layer "F.Cu") (net 15))
   (segment (start 96.8625 58.8025) (end 95.54 57.48) (width 0.25) (layer "F.Cu") (net 15))
+  (segment (start 103.25 66) (end 101.2 63.95) (width 0.25) (layer "F.Cu") (net 15))
   (segment (start 97.5 60.25) (end 96.8625 60.25) (width 0.25) (layer "F.Cu") (net 15))
   (segment (start 107.1375 66) (end 107.1375 66.65) (width 0.25) (layer "F.Cu") (net 15))
-  (segment (start 103.25 66) (end 101.2 63.95) (width 0.25) (layer "F.Cu") (net 15))
-  (segment (start 112.8625 64.05) (end 112.8625 64.7) (width 0.25) (layer "F.Cu") (net 15))
-  (via (at 105.8 66) (size 0.8) (drill 0.4) (layers "F.Cu" "B.Cu") (net 15))
+  (via (at 105.275 66) (size 0.8) (drill 0.4) (layers "F.Cu" "B.Cu") (net 15))
   (via (at 98.05 60.8) (size 0.8) (drill 0.4) (layers "F.Cu" "B.Cu") (net 15))
   (via (at 101.2 63.95) (size 0.8) (drill 0.4) (layers "F.Cu" "B.Cu") (net 15))
-  (via (at 110.4755 65.3245) (size 0.8) (drill 0.4) (layers "F.Cu" "B.Cu") (net 15))
-  (segment (start 109.8 66) (end 110.4755 65.3245) (width 0.25) (layer "B.Cu") (net 15))
   (segment (start 98.05 60.8) (end 101.2 63.95) (width 0.25) (layer "B.Cu") (net 15))
-  (segment (start 105.8 66) (end 109.8 66) (width 0.25) (layer "B.Cu") (net 15))
   (zone (net 11) (net_name "GND1") (layer "F.Cu") (name "FRONTFILL") (hatch edge 0.508)
     (connect_pads (clearance 0.508))

Commit message: updates
Connections:
- R2 pad 2: P13 -> P12
- U1 pad 13: P13 -> P12
- U1 pad 3: P13 -> P12
Routing:
- net P13: track 15.4 -> 0.00 mm, vias 2 -> 0
- net P12: track 0.00 -> 15.4 mm, vias 0 -> 2
- net GND1: track 18.7 -> 27.4 mm, vias 25 -> 27
