File: siox.kicad_sch (KiCad schematic)
At the start: 1 part, among them U1 MSP430G2131IN14

Commit message: fixes
Parts:
- added C1, C2: 0.1uF, Capacitor_SMD:C_0805_2012Metric, symbol Device:C_Small
- added J1: CE, TestPoint:TestPoint_Pad_D2.0mm, symbol Connector:Conn_01x01_Male
- added J10: M7, TestPoint:TestPoint_Pad_D2.0mm, symbol Connector:Conn_01x01_Male
- added J2: CI, TestPoint:TestPoint_Pad_D2.0mm, symbol Connector:Conn_01x01_Male
- added J3: XE, TestPoint:TestPoint_Pad_D2.0mm, symbol Connector:Conn_01x01_Male
- added J4: XI, TestPoint:TestPoint_Pad_D2.0mm, symbol Connector:Conn_01x01_Male
- added J5: M2, TestPoint:TestPoint_Pad_D2.0mm, symbol Connector:Conn_01x01_Male
- added J6: M3, TestPoint:TestPoint_Pad_D2.0mm, symbol Connector:Conn_01x01_Male
- added J7: M4, TestPoint:TestPoint_Pad_D2.0mm, symbol Connector:Conn_01x01_Male
- added J8: M5, TestPoint:TestPoint_Pad_D2.0mm, symbol Connector:Conn_01x01_Male
- added J9: M6, TestPoint:TestPoint_Pad_D2.0mm, symbol Connector:Conn_01x01_Male
- added R1: 47k, Resistor_SMD:R_0805_2012Metric, symbol Device:R_Small
- added R2, R3, R4: 10k, Resistor_SMD:R_0805_2012Metric, symbol Device:R_Small
- added U2: 12C508/9, Package_SO:SOP-8_5.28x5.23mm_P1.27mm, symbol MCU_Microchip_PIC12:PIC12F1501-IMS
- U1: value MSP430G2131IN14 -> 74HC4066
Connections:
- net CE: now reaches U1.1 (DVCC)
- net CE: now also J1.1 (Pin_1)
- net CI: now reaches U1.10 (~{RST}/NMI/SBWTDIO)
- net CI: now also U1.9 (TDI/TDO/SDI/SDA/P1.7), J2.1 (Pin_1), R4.1
- net XI: now reaches U1.11 (SBWTCK/TEST)
- net XI: now also J4.1 (Pin_1)
- net P12: now reaches U1.12 (P2.7/XOUT)
- net P12: now also U1.13 (P2.6/XIN/TA0.1), U1.5 (ADC10CLK/VREF-/VeREF-/A3/P1.3), U1.6 (TCK/SMCLK/VREF+/VeREF+/A4/P1.4), R1.1
- net +3.3V: now reaches U1.14 (DVSS)
- net +3.3V: now also C1.2, C2.1, R2.1, R3.2, R4.2, U2.1 (VDD)
- net XE: now reaches U1.2 (ACLK/TACLK/A0/P1.0)
- net XE: now also J3.1 (Pin_1), R3.1
- net P3: now reaches U1.3 (TA0.0/A1/P1.1)
- net P3: now also R2.2
- net GND1: now reaches U1.4 (TA0.1/A2/P1.2)
- net GND1: now also U1.7 (TMS/SCLK/TA0.0/A5/P1.5), C1.1, C2.2, R1.2, U2.8 (VSS)
- net PI: now reaches U1.8 (TDI/SDO/SCL/TCLK/TA0.1/P1.6)
- new net MP2: J5.1 (Pin_1), U2.2 (RA5)
- new net MP3: J6.1 (Pin_1), U2.3 (RA4)
- new net MP4: J7.1 (Pin_1), U2.4 (RA3)
- new net MP5: J8.1 (Pin_1), U2.5 (RA2)
- new net MP6: J9.1 (Pin_1), U2.6 (RA1)
- new net MP7: J10.1 (Pin_1), U2.7 (RA0)
Other:
- moved on the sheet: U1

Commit message: fix pads
Parts:
- added J11: IO_GND_1, PsioPin:PsioPin, symbol Connector:Conn_01x01_Male
- added J12: IO_GND_2, PsioPin:PsioPin, symbol Connector:Conn_01x01_Male
- added J13: IO_GND_3, PsioPin:PsioPin, symbol Connector:Conn_01x01_Male
- added J14: IO_GND_4, PsioPin:PsioPin, symbol Connector:Conn_01x01_Male
- added J15: IO_CE, PsioPin:PsioPin, symbol Connector:Conn_01x01_Male
- added J16, J19: IO_PI, PsioPin:PsioPin, symbol Connector:Conn_01x01_Male
- added J17, J18: M7, PsioPin:PsioPin, symbol Connector:Conn_01x01_Male
Connections:
- net +3.3V: now also J17.1 (Pin_1), J18.1 (Pin_1)
- net CE: now also J15.1 (Pin_1)
- net GND1: now also J11.1 (Pin_1), J12.1 (Pin_1), J13.1 (Pin_1), J14.1 (Pin_1)
- net PI: now also J16.1 (Pin_1)
- net P12 renamed EN
- net EN: now also J19.1 (Pin_1)

Commit message: updates
Parts:
- J15: value IO_CE -> IO_PE
Changed lines of the file:
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@@
-    )
-  )
-  (global_label "PE" (shape input) (at 45.085 146.685 0) (fields_autoplaced)
-    (effects (font (size 1.27 1.27)) (justify left))
-    (property "Intersheetrefs" "${INTERSHEET_REFS}" (at 45.085 148.8758 0)
-      (effects (font (size 1.27 1.27)) (justify left) hide)
     )
   )
@@
     )
   )
+  (global_label "CE" (shape input) (at 109.22 186.69 0) (fields_autoplaced)
+    (effects (font (size 1.27 1.27)) (justify left))
+    (property "Intersheetrefs" "${INTERSHEET_REFS}" (at 109.22 188.8808 0)
+      (effects (font (size 1.27 1.27)) (justify left) hide)
+    )
+  )
   (global_label "MP3" (shape input) (at 139.7 82.55 0) (fields_autoplaced)
     (effects (font (size 1.27 1.27)) (justify left))
@@
     )
   )
-  (global_label "PI" (shape input) (at 45.085 144.145 0) (fields_autoplaced)
-    (effects (font (size 1.27 1.27)) (justify left))
-    (property "Intersheetrefs" "${INTERSHEET_REFS}" (at 45.085 146.3358 0)
-      (effects (font (size 1.27 1.27)) (justify left) hide)
-    )
-  )
   (global_label "XE" (shape input) (at 138.43 31.75 180) (fields_autoplaced)
     (effects (font (size 1.27 1.27)) (justify right))
@@
     (effects (font (size 1.27 1.27)) (justify left))
     (property "Intersheetrefs" "${INTERSHEET_REFS}" (at 77.6165 50.165 0)
-      (effects (font (size 1.27 1.27)) (justify left) hide)
-    )
-  )
-  (global_label "CE" (shape input) (at 109.22 186.69 0) (fields_autoplaced)
-    (effects (font (size 1.27 1.27)) (justify left))
-    (property "Intersheetrefs" "${INTERSHEET_REFS}" (at 109.22 188.8808 0)
       (effects (font (size 1.27 1.27)) (justify left) hide)
     )
@@
   (symbol (lib_id "Power:GND1") (at 113.03 176.53 0) (mirror y) (unit 1)
     (in_bom yes) (on_board yes) (dnp no)
-    (property "Reference" "#PWR0105" (at 113.03 182.88 0)
+    (property "Reference" "#PWR0109" (at 113.03 182.88 0)
       (effects (font (size 1.27 1.27)) hide)
     )
@@
       (project "siox"
         (path "/164db33b-1b1e-4bd8-ba69-9a6e1ab7c087"
-          (reference "#PWR0105") (unit 1) (value "GND1") (footprint "")
+          (reference "#PWR0109") (unit 1) (value "GND1") (footprint "")
         )
       )
@@
       (effects (font (size 1.27 1.27)))
     )
-    (property "Value" "IO_CE" (at 98.425 185.5439 0)
+    (property "Value" "IO_PE" (at 98.425 185.5439 0)
       (effects (font (size 1.27 1.27)))
     )
@@
       (project "siox"
         (path "/164db33b-1b1e-4bd8-ba69-9a6e1ab7c087"
-          (reference "J15") (unit 1) (value "IO_CE") (footprint "PsioPin:PsioPin")
-        )
-      )
+          (reference "J15") (unit 1) (value "IO_PE") (footprint "PsioPin:PsioPin")
+        )
+      )

Commit message: updates
Connections:
- net EN: no longer U1.12 (P2.7/XOUT), U1.13 (P2.6/XIN/TA0.1)
- net P3 renamed P13
- net P13: now also U1.13 (P2.6/XIN/TA0.1)
- new net P12: U1.12 (P2.7/XOUT)
Changed lines of the file:
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@@
 (kicad_sch (version 20221110) (generator eeschema)
   (paper "A4")
+  (junction (at 180.34 26.67) (diameter 0) (color 0 0 0 0)
+  )
   (junction (at 106.68 31.115) (diameter 0) (color 0 0 0 0)
   )
   (junction (at 121.92 31.115) (diameter 0) (color 0 0 0 0)
   )
+  (junction (at 24.13 55.245) (diameter 0) (color 0 0 0 0)
+  )
   (junction (at 171.45 35.56) (diameter 0) (color 0 0 0 0)
   )
@@
     (stroke (width 0) (type default))
   )
+  (wire (pts (xy 180.34 26.67) (xy 180.34 29.21))
+    (stroke (width 0) (type default))
+  )
   (wire (pts (xy 133.35 92.71) (xy 139.7 92.71))
     (stroke (width 0) (type default))
@@
     (stroke (width 0) (type default))
   )
+  (wire (pts (xy 24.13 55.245) (xy 24.13 57.15))
+    (stroke (width 0) (type default))
+  )
   (wire (pts (xy 107.315 65.405) (xy 109.855 65.405))
     (stroke (width 0) (type default))
@@
     (stroke (width 0) (type default))
   )
+  (wire (pts (xy 180.34 29.21) (xy 182.245 29.21))
+    (stroke (width 0) (type default))
+  )
+  (wire (pts (xy 180.34 26.67) (xy 180.34 24.13))
+    (stroke (width 0) (type default))
+  )
   (wire (pts (xy 88.9 37.465) (xy 88.9 45.085))
     (stroke (width 0) (type default))
@@
     (stroke (width 0) (type default))
   )
+  (wire (pts (xy 22.86 57.15) (xy 24.13 57.15))
+    (stroke (width 0) (type default))
+  )
   (wire (pts (xy 107.315 60.325) (xy 109.855 60.325))
     (stroke (width 0) (type default))
@@
     (stroke (width 0) (type default))
   )
+  (wire (pts (xy 182.245 26.67) (xy 180.34 26.67))
+    (stroke (width 0) (type default))
+  )
   (wire (pts (xy 109.22 166.37) (xy 109.22 171.45))
     (stroke (width 0) (type default))
@@
     (stroke (width 0) (type default))
   )
+  (wire (pts (xy 22.86 57.15) (xy 22.86 55.88))
+    (stroke (width 0) (type default))
+  )
   (wire (pts (xy 133.35 97.79) (xy 139.7 97.79))
     (stroke (width 0) (type default))
@@
     (stroke (width 0) (type default))
   )
-  (wire (pts (xy 172.72 26.67) (xy 175.26 26.67))
+  (wire (pts (xy 172.72 26.67) (xy 180.34 26.67))
     (stroke (width 0) (type default))
   )
@@
     (stroke (width 0) (type default))
   )
+  (wire (pts (xy 180.34 24.13) (xy 182.88 24.13))
+    (stroke (width 0) (type default))
+  )
   (wire (pts (xy 106.045 86.36) (xy 112.395 86.36))
     (stroke (width 0) (type default))
@@
     (stroke (width 0) (type default))
   )
+  (wire (pts (xy 24.13 54.61) (xy 24.13 55.245))
+    (stroke (width 0) (type default))
+  )
   (wire (pts (xy 109.855 60.325) (xy 109.855 57.785))
     (stroke (width 0) (type default))
@@
     )
   )
-  (global_label "P3" (shape input) (at 175.26 26.67 0) (fields_autoplaced)
-    (effects (font (size 1.27 1.27)) (justify left))
-    (property "Intersheetrefs" "${INTERSHEET_REFS}" (at 180.4865 26.67 0)
+  (global_label "P3" (shape input) (at 182.245 29.21 0) (fields_autoplaced)
+    (effects (font (size 1.27 1.27)) (justify left))
+    (property "Intersheetrefs" "${INTERSHEET_REFS}" (at 188.7415 29.21 0)
       (effects (font (size 1.27 1.27)) (justify left) hide)
     )
@@
     )
   )
-  (global_label "EN" (shape input) (at 24.13 55.245 180) (fields_autoplaced)
-    (effects (font (size 1.27 1.27)) (justify right))
-    (property "Intersheetrefs" "${INTERSHEET_REFS}" (at 18.9035 55.245 0)
-      (effects (font (size 1.27 1.27)) (justify right) hide)
-    )
-  )
   (global_label "P5" (shape input) (at 107.315 57.785 180) (fields_autoplaced)
     (effects (font (size 1.27 1.27)) (justify right))
@@
     )
   )
-  (global_label "P13" (shape input) (at 107.315 65.405 180) (fields_autoplaced)
-    (effects (font (size 1.27 1.27)) (justify right))
-    (property "Intersheetrefs" "${INTERSHEET_REFS}" (at 107.315 67.5958 0)
-      (effects (font (size 1.27 1.27)) (justify right) hide)
+  (global_label "P13" (shape input) (at 182.245 26.67 0) (fields_autoplaced)
+    (effects (font (size 1.27 1.27)) (justify left))
+    (property "Intersheetrefs" "${INTERSHEET_REFS}" (at 180.975 28.8608 0)
+      (effects (font (size 1.27 1.27)) (justify left) hide)
     )
   )
@@
     )
   )
+  (global_label "P13" (shape input) (at 182.88 24.13 0) (fields_autoplaced)
+    (effects (font (size 1.27 1.27)) (justify left))
+    (property "Intersheetrefs" "${INTERSHEET_REFS}" (at 181.61 26.3208 0)
+      (effects (font (size 1.27 1.27)) (justify left) hide)
+    )
+  )
   (global_label "MP2" (shape input) (at 63.5 86.995 0) (fields_autoplaced)
     (effects (font (size 1.27 1.27)) (justify left))
@@
       (effects (font (size 1.27 1.27)) (justify right) hide)
     )
+  )
+  (global_label "P12" (shape input) (at 22.86 55.88 180) (fields_autoplaced)
+    (effects (font (size 1.27 1.27)) (justify right))
+    (property "Intersheetrefs" "${INTERSHEET_REFS}" (at 22.86 58.0708 0)
+      (effects (font (size 1.27 1.27)) (justify right) hide)
+    )

Commit message: updates
Connections:
- net P13 is gone; now on net P12: R2.2, U1.13 (P2.6/XIN/TA0.1), U1.3 (TA0.0/A1/P1.1)
Changed lines of the file:
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@@
   (junction (at 121.92 31.115) (diameter 0) (color 0 0 0 0)
   )
-  (junction (at 24.13 55.245) (diameter 0) (color 0 0 0 0)
-  )
   (junction (at 171.45 35.56) (diameter 0) (color 0 0 0 0)
   )
@@
     (stroke (width 0) (type default))
   )
-  (wire (pts (xy 24.13 55.245) (xy 24.13 57.15))
-    (stroke (width 0) (type default))
-  )
   (wire (pts (xy 107.315 65.405) (xy 109.855 65.405))
     (stroke (width 0) (type default))
@@
     (stroke (width 0) (type default))
   )
+  (wire (pts (xy 24.13 54.61) (xy 24.13 55.245))
+    (stroke (width 0) (type default))
+  )
   (wire (pts (xy 171.45 35.56) (xy 175.26 35.56))
     (stroke (width 0) (type default))
@@
     (stroke (width 0) (type default))
   )
-  (wire (pts (xy 22.86 57.15) (xy 24.13 57.15))
-    (stroke (width 0) (type default))
-  )
   (wire (pts (xy 107.315 60.325) (xy 109.855 60.325))
     (stroke (width 0) (type default))
@@
     (stroke (width 0) (type default))
   )
-  (wire (pts (xy 22.86 57.15) (xy 22.86 55.88))
-    (stroke (width 0) (type default))
-  )
   (wire (pts (xy 133.35 97.79) (xy 139.7 97.79))
     (stroke (width 0) (type default))
@@
     (stroke (width 0) (type default))
   )
+  (wire (pts (xy 21.59 54.61) (xy 24.13 54.61))
+    (stroke (width 0) (type default))
+  )
   (wire (pts (xy 106.045 86.36) (xy 112.395 86.36))
     (stroke (width 0) (type default))
@@
     (stroke (width 0) (type default))
   )
-  (wire (pts (xy 24.13 54.61) (xy 24.13 55.245))
-    (stroke (width 0) (type default))
-  )
   (wire (pts (xy 109.855 60.325) (xy 109.855 57.785))
     (stroke (width 0) (type default))
@@
     )
   )
-  (global_label "P13" (shape input) (at 182.88 24.13 0) (fields_autoplaced)
-    (effects (font (size 1.27 1.27)) (justify left))
-    (property "Intersheetrefs" "${INTERSHEET_REFS}" (at 181.61 26.3208 0)
+  (global_label "P12" (shape input) (at 182.88 24.13 0) (fields_autoplaced)
+    (effects (font (size 1.27 1.27)) (justify left))
+    (property "Intersheetrefs" "${INTERSHEET_REFS}" (at 182.88 26.3208 0)
       (effects (font (size 1.27 1.27)) (justify left) hide)
     )
@@
     )
   )
+  (global_label "P12" (shape input) (at 21.59 54.61 180) (fields_autoplaced)
+    (effects (font (size 1.27 1.27)) (justify right))
+    (property "Intersheetrefs" "${INTERSHEET_REFS}" (at 15.154 54.61 0)
+      (effects (font (size 1.27 1.27)) (justify right) hide)
+    )
+  )
   (global_label "P14" (shape input) (at 120.65 27.305 180) (fields_autoplaced)
     (effects (font (size 1.27 1.27)) (justify right))
@@
       (effects (font (size 1.27 1.27)) (justify right) hide)
     )
-  )
-  (global_label "P12" (shape input) (at 22.86 55.88 180) (fields_autoplaced)
-    (effects (font (size 1.27 1.27)) (justify right))
-    (property "Intersheetrefs" "${INTERSHEET_REFS}" (at 22.86 58.0708 0)
-      (effects (font (size 1.27 1.27)) (justify right) hide)
-    )
